Commit message: finished assignment

File: body.urdf (robot description, URDF)
Before this commit: robot robot, 3 links, 2 joints
Joints:
- joint Torso_BackLeg: origin xyz=0 1.0 0 rpy=0 0 0 -> xyz=1 0 1 rpy=0 0 0
- joint Torso_FrontLeg: origin xyz=0 -0.5 -0.5 rpy=0 0 0 -> xyz=2 0 1 rpy=0 0 0

Commit message: End of task 4

File: body.urdf (robot description, URDF)
Before this commit: robot robot, 3 links, 2 joints
Links:
- added link BackLowerLeg, mass 1; collision box size=0.2 0.2 1; visual box size=0.2 0.2 1
- added link FrontLowerLeg, mass 1; collision box size=0.2 0.2 1; visual box size=0.2 0.2 1
- added link LeftLeg, mass 1; collision box size=1 0.2 0.2; visual box size=1 0.2 0.2
- added link LeftLowerLeg, mass 1; collision box size=0.2 0.2 1; visual box size=0.2 0.2 1
- added link RightLeg, mass 1; collision box size=1 0.2 0.2; visual box size=1 0.2 0.2
- added link RightLowerLeg, mass 1; collision box size=0.2 0.2 1; visual box size=0.2 0.2 1
- link BackLeg: geometry collision box size=0.2 1 0.2; visual box size=0.2 1 0.2
- link FrontLeg: geometry collision box size=0.2 1 0.2; visual box size=0.2 1 0.2
Joints:
- added joint BackLeg_BackLowerLeg: type revolute, parent BackLeg, child BackLowerLeg, origin xyz=0 -1 0 rpy=0 0 0, axis 1 0 0, limit lower=-3.14159 upper=3.14159 effort=0.0 velocity=0.0
- added joint FrontLeg_FrontLowerLeg: type revolute, parent FrontLeg, child FrontLowerLeg, origin xyz=0 1 0 rpy=0 0 0, axis 1 0 0, limit lower=-3.14159 upper=3.14159 effort=0.0 velocity=0.0
- added joint LeftLeg_LeftLowerLeg: type revolute, parent LeftLeg, child LeftLowerLeg, origin xyz=1 0 0 rpy=0 0 0, axis 0 1 0, limit lower=-3.14159 upper=3.14159 effort=0.0 velocity=0.0
- added joint RightLeg_RightLowerLeg: type revolute, parent RightLeg, child RightLowerLeg, origin xyz=-1 0 0 rpy=0 0 0, axis 0 1 0, limit lower=-3.14159 upper=3.14159 effort=0.0 velocity=0.0
- added joint Torso_LeftLeg: type revolute, parent Torso, child LeftLeg, origin xyz=0.5 0 1 rpy=0 0 0, axis 0 1 0, limit lower=-3.14159 upper=3.14159 effort=0.0 velocity=0.0
- added joint Torso_RightLeg: type revolute, parent Torso, child RightLeg, origin xyz=-0.5 0 1 rpy=0 0 0, axis 0 1 0, limit lower=-3.14159 upper=3.14159 effort=0.0 velocity=0.0
- joint Torso_BackLeg: axis 0 1 0 -> 1 0 0; origin xyz=1 0 1 rpy=0 0 0 -> xyz=0 -0.5 1 rpy=0 0 0
- joint Torso_FrontLeg: axis 0 1 0 -> 1 0 0; origin xyz=2 0 1 rpy=0 0 0 -> xyz=0 0.5 1 rpy=0 0 0

Commit message: octoped

File: body.urdf (robot description, URDF)
Before this commit: robot robot, 9 links, 8 joints
Links:
- added link BackLegv2, mass 1; collision box size=0.2 1 0.2; visual box size=0.2 1 0.2
- added link BackLowerLegv2, mass 1; collision box size=0.2 0.2 1; visual box size=0.2 0.2 1
- added link FrontLegv2, mass 1; collision box size=0.2 1 0.2; visual box size=0.2 1 0.2
- added link FrontLowerLegv2, mass 1; collision box size=0.2 0.2 1; visual box size=0.2 0.2 1
- added link LeftLegv2, mass 1; collision box size=1 0.2 0.2; visual box size=1 0.2 0.2
- added link LeftLowerLegv2, mass 1; collision box size=0.2 0.2 1; visual box size=0.2 0.2 1
- added link RightLegv2, mass 1; collision box size=1 0.2 0.2; visual box size=1 0.2 0.2
- added link RightLowerLegv2, mass 1; collision box size=0.2 0.2 1; visual box size=0.2 0.2 1
Joints:
- added joint BackLeg_BackLowerLegv2: type revolute, parent BackLegv2, child BackLowerLegv2, origin xyz=-0.125 -1 0 rpy=0 0 0, axis 1 0 0, limit lower=-3.14159 upper=3.14159 effort=0.0 velocity=0.0
- added joint FrontLeg_FrontLowerLegv2: type revolute, parent FrontLegv2, child FrontLowerLegv2, origin xyz=-0.125 1 0 rpy=0 0 0, axis 1 0 0, limit lower=-3.14159 upper=3.14159 effort=0.0 velocity=0.0
- added joint LeftLeg_LeftLowerLegv2: type revolute, parent LeftLegv2, child LeftLowerLegv2, origin xyz=1 -0.125 0 rpy=0 0 0, axis 0 1 0, limit lower=-3.14159 upper=3.14159 effort=0.0 velocity=0.0
- added joint RightLeg_RightLowerLegv2: type revolute, parent RightLegv2, child RightLowerLegv2, origin xyz=-1 -0.125 0 rpy=0 0 0, axis 0 1 0, limit lower=-3.14159 upper=3.14159 effort=0.0 velocity=0.0
- added joint Torso_BackLegv2: type revolute, parent Torso, child BackLegv2, origin xyz=-0.125 -0.5 1 rpy=0 0 0, axis 1 0 0, limit lower=-3.14159 upper=3.14159 effort=0.0 velocity=0.0
- added joint Torso_FrontLegv2: type revolute, parent Torso, child FrontLegv2, origin xyz=-0.125 0.5 1 rpy=0 0 0, axis 1 0 0, limit lower=-3.14159 upper=3.14159 effort=0.0 velocity=0.0
- added joint Torso_LeftLegv2: type revolute, parent Torso, child LeftLegv2, origin xyz=0.5 -0.125 1 rpy=0 0 0, axis 0 1 0, limit lower=-3.14159 upper=3.14159 effort=0.0 velocity=0.0
- added joint Torso_RightLegv2: type revolute, parent Torso, child RightLegv2, origin xyz=-0.5 -0.125 1 rpy=0 0 0, axis 0 1 0, limit lower=-3.14159 upper=3.14159 effort=0.0 velocity=0.0
- joint BackLeg_BackLowerLeg: origin xyz=0 -1 0 rpy=0 0 0 -> xyz=0.125 -1 0 rpy=0 0 0
- joint FrontLeg_FrontLowerLeg: origin xyz=0 1 0 rpy=0 0 0 -> xyz=0.125 1 0 rpy=0 0 0
- joint LeftLeg_LeftLowerLeg: origin xyz=1 0 0 rpy=0 0 0 -> xyz=1 0.125 0 rpy=0 0 0
- joint RightLeg_RightLowerLeg: origin xyz=-1 0 0 rpy=0 0 0 -> xyz=-1 0.125 0 rpy=0 0 0
- joint Torso_BackLeg: origin xyz=0 -0.5 1 rpy=0 0 0 -> xyz=0.125 -0.5 1 rpy=0 0 0
- joint Torso_FrontLeg: origin xyz=0 0.5 1 rpy=0 0 0 -> xyz=0.125 0.5 1 rpy=0 0 0
- joint Torso_LeftLeg: origin xyz=0.5 0 1 rpy=0 0 0 -> xyz=0.5 0.125 1 rpy=0 0 0
- joint Torso_RightLeg: origin xyz=-0.5 0 1 rpy=0 0 0 -> xyz=-0.5 0.125 1 rpy=0 0 0

Commit message: Assignment 6

File: body.urdf (robot description, URDF)
Before this commit: robot robot, 17 links, 16 joints
Links:
- removed link BackLeg
- removed link BackLegv2
- removed link BackLowerLeg
- removed link BackLowerLegv2
- removed link FrontLeg
- removed link FrontLegv2
- removed link FrontLowerLeg
- removed link FrontLowerLegv2
- removed link LeftLeg
- removed link LeftLegv2
- removed link LeftLowerLeg
- removed link LeftLowerLegv2
- removed link RightLeg
- removed link RightLegv2
- removed link RightLowerLeg
- removed link RightLowerLegv2
- removed link Torso
- added link Cube0, mass 1; collision box size=1 1 1; visual box size=1 1 1
- added link Cube1, mass 1; collision box size=1 1 2; visual box size=1 1 2
- added link Cube2, mass 1; collision box size=1 1 1; visual box size=1 1 1
- added link Cube3, mass 1; collision box size=1 1 1; visual box size=1 1 1
- added link Cube4, mass 1; collision box size=1 2 2; visual box size=1 2 2
- added link Cube5, mass 1; collision box size=1 1 2; visual box size=1 1 2
- added link Cube6, mass 1; collision box size=1 2 1; visual box size=1 2 1
Joints:
- removed joint BackLeg_BackLowerLeg
- removed joint BackLeg_BackLowerLegv2
- removed joint FrontLeg_FrontLowerLeg
- removed joint FrontLeg_FrontLowerLegv2
- removed joint LeftLeg_LeftLowerLeg
- removed joint LeftLeg_LeftLowerLegv2
- removed joint RightLeg_RightLowerLeg
- removed joint RightLeg_RightLowerLegv2
- removed joint Torso_BackLeg
- removed joint Torso_BackLegv2
- removed joint Torso_FrontLeg
- removed joint Torso_FrontLegv2
- removed joint Torso_LeftLeg
- removed joint Torso_LeftLegv2
- removed joint Torso_RightLeg
- removed joint Torso_RightLegv2
- added joint Joint_Cube0_Cube1: type revolute, parent Cube0, child Cube1, origin xyz=0.5 0 0.5 rpy=0 0 0, axis 0 1 0, limit lower=-3.14159 upper=3.14159 effort=0.0 velocity=0.0
- added joint Joint_Cube1_Cube2: type revolute, parent Cube1, child Cube2, origin xyz=1 0 0 rpy=0 0 0, axis 0 1 0, limit lower=-3.14159 upper=3.14159 effort=0.0 velocity=0.0
- added joint Joint_Cube2_Cube3: type revolute, parent Cube2, child Cube3, origin xyz=1 0 0 rpy=0 0 0, axis 0 1 0, limit lower=-3.14159 upper=3.14159 effort=0.0 velocity=0.0
- added joint Joint_Cube3_Cube4: type revolute, parent Cube3, child Cube4, origin xyz=1 0 0 rpy=0 0 0, axis 0 1 0, limit lower=-3.14159 upper=3.14159 effort=0.0 velocity=0.0
- added joint Joint_Cube4_Cube5: type revolute, parent Cube4, child Cube5, origin xyz=1 0 0 rpy=0 0 0, axis 0 1 0, limit lower=-3.14159 upper=3.14159 effort=0.0 velocity=0.0
- added joint Joint_Cube5_Cube6: type revolute, parent Cube5, child Cube6, origin xyz=1 0 0 rpy=0 0 0, axis 0 1 0, limit lower=-3.14159 upper=3.14159 effort=0.0 velocity=0.0

Commit message: assignment 6 review

File: body.urdf (robot description, URDF)
Before this commit: robot robot, 7 links, 6 joints
Links:
- removed link Cube4
- removed link Cube5
- removed link Cube6
- link Cube0: geometry collision box size=0.26837121767644656 0.3294055604764292 0.21791903675394964; visual box size=0.26837121767644656 0.3294055604764292 0.21791903675394964
- link Cube1: geometry collision box size=0.33953643992725546 0.19154473814974765 0.14985584372786614; visual box size=0.33953643992725546 0.19154473814974765 0.14985584372786614
- link Cube2: geometry collision box size=0.2578979545166123 0.28120607499198114 0.34578198841434526; visual box size=0.2578979545166123 0.28120607499198114 0.34578198841434526
- link Cube3: geometry collision box size=0.1699540707659037 0.14933516278266917 0.15948665405488835; visual box size=0.1699540707659037 0.14933516278266917 0.15948665405488835
Joints:
- removed joint Joint_Cube0_Cube1
- removed joint Joint_Cube1_Cube2
- removed joint Joint_Cube2_Cube3
- removed joint Joint_Cube3_Cube4
- removed joint Joint_Cube4_Cube5
- removed joint Joint_Cube5_Cube6
- added joint Cube0_Cube1: type revolute, parent Cube0, child Cube1, origin xyz=0.13418560883822328 0 0.5 rpy=0 0 0, axis 0 0 1, limit lower=-3.14159 upper=3.14159 effort=0.0 velocity=0.0
- added joint Cube1_Cube2: type revolute, parent Cube1, child Cube2, origin xyz=0.33953643992725546 0 0 rpy=0 0 0, axis 0 0 1, limit lower=-3.14159 upper=3.14159 effort=0.0 velocity=0.0
- added joint Cube2_Cube3: type revolute, parent Cube2, child Cube3, origin xyz=0.2578979545166123 0 0 rpy=0 0 0, axis 0 0 1, limit lower=-3.14159 upper=3.14159 effort=0.0 velocity=0.0

Commit message: Assignment7

File: body.urdf (robot description, URDF)
Before this commit: robot robot, 4 links, 3 joints
Links:
- link Cube0: geometry collision box size=0.2 0.2 0.2; visual box size=0.2 0.2 0.2
- link Cube1: geometry collision box size=0.18987154223080027 0.23340323113024378 0.19630358648824864; visual box size=0.18987154223080027 0.23340323113024378 0.19630358648824864
- link Cube2: geometry collision box size=0.21971498998419897 0.13648442095997362 0.17067586890017827; visual box size=0.21971498998419897 0.13648442095997362 0.17067586890017827
- link Cube3: geometry collision box size=0.11244343826818916 0.22491340411461372 0.3776988841860053; visual box size=0.11244343826818916 0.22491340411461372 0.3776988841860053
Joints:
- removed joint Cube1_Cube2
- removed joint Cube2_Cube3
- added joint Cube0_Cube2: type revolute, parent Cube0, child Cube2, origin xyz=-0.1 0 0.5 rpy=0 0 0, axis 0 0 1, limit lower=-3.14159 upper=3.14159 effort=0.0 velocity=0.0
- added joint Cube0_Cube3: type revolute, parent Cube0, child Cube3, origin xyz=0 0.1 0.5 rpy=0 0 0, axis 0 0 1, limit lower=-3.14159 upper=3.14159 effort=0.0 velocity=0.0
- joint Cube0_Cube1: origin xyz=0.13418560883822328 0 0.5 rpy=0 0 0 -> xyz=0.1 0 0.5 rpy=0 0 0

Commit message: assignment 7

File: body.urdf (robot description, URDF)
Before this commit: robot robot, 4 links, 3 joints
Links:
- added link Cube4, mass 1; collision box size=0.3674765229050103 0.36571814407165726 0.30336701884895567; visual box size=0.3674765229050103 0.36571814407165726 0.30336701884895567
- added link Cube5, mass 1; collision box size=0.2668254622182148 0.14409119946317422 0.3744017980439003; visual box size=0.2668254622182148 0.14409119946317422 0.3744017980439003
- added link Cube6, mass 1; collision box size=0.2 0.32026085216563216 0.280549821740053; visual box size=0.2 0.32026085216563216 0.280549821740053
- link Cube1: geometry collision box size=0.21662397255684013 0.2 0.29027787578887276; visual box size=0.21662397255684013 0.2 0.29027787578887276
- link Cube2: geometry collision box size=0.17748704573014235 0.2835193909088872 0.23904230847265132; visual box size=0.17748704573014235 0.2835193909088872 0.23904230847265132
- link Cube3: geometry collision box size=0.23611956663191833 0.1621295737739487 0.18292275000288968; visual box size=0.23611956663191833 0.1621295737739487 0.18292275000288968
Joints:
- added joint Cube0_Cube4: type revolute, parent Cube0, child Cube4, origin xyz=0 -0.1 0.5 rpy=0 0 0, axis 0 0 1, limit lower=-3.14159 upper=3.14159 effort=0.0 velocity=0.0
- added joint Cube0_Cube5: type revolute, parent Cube0, child Cube5, origin xyz=0 0 0.6 rpy=0 0 0, axis 0 0 1, limit lower=-3.14159 upper=3.14159 effort=0.0 velocity=0.0
- added joint Cube1_Cube6: type revolute, parent Cube1, child Cube6, origin xyz=0 0.1 0 rpy=0 0 0, axis 0 0 1, limit lower=-3.14159 upper=3.14159 effort=0.0 velocity=0.0

Commit message: update to ass7

File: body.urdf (robot description, URDF)
Before this commit: robot robot, 7 links, 6 joints
Links:
- removed link Cube4
- removed link Cube5
- removed link Cube6
- link Cube1: geometry collision box size=0.3913909664123233 0.2 0.22300508805072716; visual box size=0.3913909664123233 0.2 0.22300508805072716
- link Cube2: geometry collision box size=0.1607205173825933 0.30618817736141934 0.3026644169862168; visual box size=0.1607205173825933 0.30618817736141934 0.3026644169862168
- link Cube3: geometry collision box size=0.2 0.11495657785366319 0.15748847869589472; visual box size=0.2 0.11495657785366319 0.15748847869589472
Joints:
- removed joint Cube0_Cube3
- removed joint Cube0_Cube4
- removed joint Cube0_Cube5
- removed joint Cube1_Cube6
- added joint Cube1_Cube3: type revolute, parent Cube1, child Cube3, origin xyz=0 0.1 0 rpy=0 0 0, axis 0 0 1, limit lower=-3.14159 upper=3.14159 effort=0.0 velocity=0.0
