Commit message: best so far

File: body31.urdf (robot description, URDF)
Before this commit: robot robot, 4 links, 3 joints
Links:
- added link Cube4, mass 1; collision box size=0.14387606914764992 0.1956371888969107 0.12656967340665418; visual box size=0.14387606914764992 0.1956371888969107 0.12656967340665418
- added link Cube5, mass 1; collision box size=0.2 0.37198716878615057 0.3852002488800568; visual box size=0.2 0.37198716878615057 0.3852002488800568
- link Cube1: geometry collision box size=0.2784289711563771 0.2 0.1331715459748355; visual box size=0.2784289711563771 0.2 0.1331715459748355
- link Cube2: geometry collision box size=0.35222953469720153 0.2110196991660159 0.18940900428732302; visual box size=0.35222953469720153 0.2110196991660159 0.18940900428732302
- link Cube3: geometry collision box size=0.110858461875385 0.34576742193721305 0.32192771585251645; visual box size=0.110858461875385 0.34576742193721305 0.32192771585251645
Joints:
- removed joint Cube1_Cube3
- added joint Cube0_Cube3: type revolute, parent Cube0, child Cube3, origin xyz=0 0.1 0.5 rpy=0 0 0, axis 0 0 1, limit lower=-3.14159 upper=3.14159 effort=0.0 velocity=0.0
- added joint Cube0_Cube4: type revolute, parent Cube0, child Cube4, origin xyz=0 -0.1 0.5 rpy=0 0 0, axis 0 0 1, limit lower=-3.14159 upper=3.14159 effort=0.0 velocity=0.0
- added joint Cube1_Cube5: type revolute, parent Cube1, child Cube5, origin xyz=0 0.1 0 rpy=0 0 0, axis 0 0 1, limit lower=-3.14159 upper=3.14159 effort=0.0 velocity=0.0
